File: hardware/ESP82_Sensor_interface.brd (EAGLE design)
At the start: 26.4 x 63.4 mm, 13 parts

Commit message: new hardware version
Parts:
- added SERIAL: (no value), SparkFun-Connectors:1X02
- added U$1, U$2: (no value), WingTechCorner:M3-HOLE
- WEMOS2: value Wemos D1 mini -> Wemos D1
- moved JST 20.4 mm to (23.7, 11.1), turned to 180 degrees
- moved R1 8.40 mm to (19.1, 45.1), turned to 0 degrees
- moved JP2 7.84 mm to (9.45, 54.0)
- moved JP1 6.81 mm to (21.6, 54.0), turned to 0 degrees
- moved BATT+ 4.35 mm to (20.0, 20.5)
- moved PIN0 4.35 mm to (20.1, 2.29)
- moved GND 4.35 mm to (6.50, 20.5)
- moved KK 4.35 mm to (6.30, 2.29)
- moved R2 3.85 mm to (16.2, 47.8)
- moved BATT 3.42 mm to (2.16, 6.09), turned to 270 degrees
- moved WEMOS1 0.56 mm to (24.5, 31.2)
- moved WEMOS2 0.56 mm to (1.59, 49.0)
Connections:
- new net RX: SERIAL.2, WEMOS2.7
- new net TX: SERIAL.1, WEMOS2.8
- net 3.3V: now also R1.1; no longer JP1.1
- net A0: now also JP1.2, R1.2; no longer R1.1
- net ENTREEGND: now also S1.2
- net GND: now also JP1.1, S1.3; no longer JP1.2, R1.2, S1.2
Routing:
- net 5V: track 67.3 -> 94.2 mm
- net TX: track 0.00 -> 24.1 mm
- net RX: track 0.00 -> 22.0 mm
- net ENTREEGND: track 22.6 -> 42.4 mm
- net D2: track 39.5 -> 27.1 mm
- net GND: track 76.5 -> 64.7 mm, vias 0 -> 1
- net 3.3V: track 26.5 -> 30.1 mm
- net A0: track 22.6 -> 24.4 mm
Other:
- board size 26.4 x 63.4 mm -> 26.4 x 58.5 mm
- board text added: "3.3V"
- board text added: "RX"
- board text added: "TX"
- board text removed: "D1"
- board text removed: "D5"
- board text removed: "D6"

Commit message: New board
Connections:
- new net N$1: JP2.2, WEMOS2.4
Routing:
- net GND: track 64.7 -> 84.7 mm
- net N$1: track 0.00 -> 16.9 mm
Other:
- board text added: "D3"
Changed lines of the file:
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@@
 <text x="5.2638375" y="50.37368125" size="1.27" layer="26" rot="R90">TX</text>
 <text x="2.7138375" y="50.22368125" size="1.27" layer="26" rot="R90">RX</text>
+<text x="3.92208125" y="40.9369625" size="1.27" layer="25">D3</text>
+<text x="12.5630375" y="50.12208125" size="1.27" layer="25" rot="R90">D3</text>
 </plain>
 <attributes>
@@
 </polygon>
 <contactref element="JP2" pad="1"/>
-<wire x1="9.45" y1="57.4" x2="22.4" y2="57.4" width="0.254" layer="16"/>
 <contactref element="JP1" pad="1"/>
-<wire x1="22.4" y1="57.4" x2="21.55" y2="54" width="0.254" layer="16"/>
 <contactref element="S1" pad="3"/>
 <wire x1="21.55" y1="54" x2="21.55" y2="51.209259375" width="0.254" layer="16"/>
@@
 <wire x1="22" y1="24.7" x2="22" y2="50.925925" width="0.254" layer="16"/>
 <wire x1="3.95" y1="15.35" x2="3.95" y2="15.9706" width="0.254" layer="1"/>
+<wire x1="1.59408125" y1="46.4449625" x2="9.14911875" y2="54" width="0.1524" layer="16"/>
+<wire x1="9.14911875" y1="54" x2="9.45" y2="54" width="0.1524" layer="16"/>
+<wire x1="9.45" y1="54" x2="9.45" y2="56.15" width="0.1524" layer="16"/>
+<wire x1="9.45" y1="56.15" x2="19.4" y2="56.15" width="0.1524" layer="16"/>
+<wire x1="19.4" y1="56.15" x2="21.55" y2="54" width="0.1524" layer="16"/>
+<wire x1="3.95" y1="15.35" x2="3.95" y2="17.54959375" width="0.1524" layer="1"/>
+<wire x1="3.95" y1="17.54959375" x2="5.2262" y2="18.82579375" width="0.1524" layer="1"/>
+<wire x1="5.2262" y1="18.82579375" x2="5.2262" y2="21.37420625" width="0.1524" layer="1"/>
+<wire x1="5.2262" y1="21.37420625" x2="3.9794" y2="22.62100625" width="0.1524" layer="1"/>
+<wire x1="3.9794" y1="22.62100625" x2="3.9794" y2="24.65" width="0.1524" layer="1"/>
 </signal>
 <signal name="N$6">
@@
 <wire x1="4.7" y1="34.31088125" x2="1.59408125" y2="31.2049625" width="0.254" layer="1"/>
 </signal>
+<signal name="N$1">
+<contactref element="WEMOS2" pad="4"/>
+<contactref element="JP2" pad="2"/>
+<wire x1="1.59408125" y1="41.3649625" x2="11.99" y2="51.76088125" width="0.254" layer="16"/>
+<wire x1="11.99" y1="51.76088125" x2="11.99" y2="54" width="0.254" layer="16"/>
+</signal>
 </signals>
