File: hardware/ESP82_Sensor_interface.sch (EAGLE design)
At the start: 14 parts

Commit message: New board
Connections:
- new net N$1: JP2.2, WEMOS2.4
Changed lines of the file:
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@@
+</segment>
+</net>
+<net name="N$1" class="0">
+<segment>
+<pinref part="WEMOS2" gate="G$1" pin="4"/>
+<wire x1="40.64" y1="43.18" x2="40.64" y2="33.02" width="0.1524" layer="91"/>
+<wire x1="40.64" y1="33.02" x2="17.78" y2="33.02" width="0.1524" layer="91"/>
+<pinref part="JP2" gate="G$1" pin="2"/>
+<wire x1="17.78" y1="33.02" x2="17.78" y2="86.36" width="0.1524" layer="91"/>
+<wire x1="17.78" y1="86.36" x2="17.78" y2="88.9" width="0.1524" layer="91"/>
+<junction x="17.78" y="86.36"/>
 </segment>
 </net>
